File: schematics/nrf24l01_pa_lna/nrf24l01_pa_lna.kicad_sch (KiCad schematic)
At the start: 44 parts, among them J1 Conn_Coaxial_Small, J2 Conn_02x04_Counter_Clockwise, U1 NRF24L01, U3 MCP1802x-xx02xOT, Y1 Crystal

Commit message: Designing the schematic and picking specific components.
Parts:
- removed J2: Conn_02x04_Counter_Clockwise, symbol Connector_Generic:Conn_02x04_Counter_Clockwise
- added C23, C24: 1u, Capacitor_SMD:C_0402_1005Metric, symbol Device:C
- added C25, C26, C27: 10n, Capacitor_SMD:C_0402_1005Metric, symbol Device:C
- added J3: Conn_02x04_Odd_Even, Connector_PinHeader_2.54mm:PinHeader_2x04_P2.54mm_Vertical, symbol Connector_Generic:Conn_02x04_Odd_Even
- C1, C10, C11, C2, C6, C7, C8, C9: footprint (none) -> Capacitor_SMD:C_0402_1005Metric; url (none) -> https://www.digikey.com/en/products/detail/yageo/CC0402KRX7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
- C12, C13: value 22p -> 18p; footprint (none) -> Capacitor_SMD:C_0402_1005Metric; url (none) -> https://www.digikey.com/en/products/detail/yageo/CC0402JRNP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
- C14, C15: footprint (none) -> Capacitor_SMD:C_0402_1005Metric; url (none) -> https://www.digikey.com/en/products/detail/yageo/CC0402KRX5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
- C16, C17, C18, C19, C20, C4: footprint (none) -> Capacitor_SMD:C_0402_1005Metric; url (none) -> https://www.digikey.com/en/products/detail/yageo/CQ0402ARNP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
- C21, C22: URL https://www.digikey.com/product-detail/en/samsung-electro-m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 -> (none); url (none) -> https://www.digikey.com/product-detail/en/samsung-electro-m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
- C3: footprint (none) -> Capacitor_SMD:C_0402_1005Metric; url (none) -> https://www.digikey.com/en/products/detail/yageo/CC0402CRNP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
- C5: footprint (none) -> Capacitor_SMD:C_0402_1005Metric; url (none) -> https://www.digikey.com/en/products/detail/yageo/CQ0402BRNP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
- J1: url (none) -> https://www.digikey.com/en/products/detail/amphenol-rf/1322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
- L1: footprint (none) -> Inductor_SMD:L_0402_1005Metric; url (none) -> https://www.digikey.com/en/products/detail/vishay-dale/ILC0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
- L2, L3, L4, L5: footprint (none) -> Inductor_SMD:L_0402_1005Metric; url (none) -> https://www.digikey.com/en/products/detail/murata-electroni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
- R1, R3, R4, R5, R6, R7: footprint (none) -> Resistor_SMD:R_0402_1005Metric; url (none) -> https://www.digikey.com/en/products/detail/yageo/AC0402JR-0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
- R10, R11, R2, R9: footprint (none) -> Resistor_SMD:R_0402_1005Metric; url (none) -> https://www.digikey.com/en/products/detail/yageo/RC0402JR-0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
- R8: footprint (none) -> Resistor_SMD:R_0402_1005Metric; url (none) -> https://www.digikey.com/en/products/detail/te-connectivity-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
- U1: url (none) -> https://www.digikey.com/en/products/detail/nordic-semicondu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
- U2: url (none) -> https://www.digikey.com/en/products/detail/skyworks-solutio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
- U3: url (none) -> https://www.digikey.com/en/products/detail/microchip-techno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
- Y1: footprint (none) -> Crystal:Crystal_HC18-U_Vertical; url (none) -> https://www.digikey.com/en/products/detail/ecs-inc/ECS-160-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
Connections:
- net GND: now also C23.2, C24.2, C25.2, C26.2, C27.2, J3.8 (Pin_8)
- net VDD: now also C23.1, C24.1, C25.1, C26.1, C27.1
- net ce: now also J3.6 (Pin_6)
- net irq: now also J3.1 (Pin_1)
- net miso: now also J3.2 (Pin_2)
- net mosi: now also J3.3 (Pin_3)
- net sck: now also J3.4 (Pin_4)
- net scn: now also J3.5 (Pin_5)
- net v_pwr: now also J3.7 (Pin_7)
Other:
- moved on the sheet: C14, C15

Commit message: Power flags to avoid KiCad errors.
Changed lines of the file:
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@@
 	(wire
 		(pts
+			(xy 109.22 113.03) (xy 109.22 115.57)
+		)
+		(stroke
+			(width 0)
+			(type default)
+		)
+	)
+	(wire
+		(pts
 			(xy 63.5 101.6) (xy 63.5 104.14)
 		)
@@
 	(wire
 		(pts
+			(xy 38.1 246.38) (xy 38.1 248.92)
+		)
+		(stroke
+			(width 0)
+			(type default)
+		)
+	)
+	(wire
+		(pts
 			(xy 82.55 140.97) (xy 82.55 133.35)
 		)
@@
 	)
 	(symbol
+		(lib_id "power:GND")
+		(at 109.22 115.57 0)
+		(unit 1)
+		(exclude_from_sim no)
+		(in_bom yes)
+		(on_board yes)
+		(dnp no)
+		(fields_autoplaced yes)
+		(property "Reference" "#PWR049"
+			(at 109.22 121.92 0)
+			(effects
+				(font
+					(size 1.27 1.27)
+				)
+				(hide yes)
+			)
+		)
+		(property "Value" "GND"
+			(at 109.22 120.65 0)
+			(effects
+				(font
+					(size 1.27 1.27)
+				)
+			)
+		)
+		(property "Footprint" ""
+			(at 109.22 115.57 0)
+			(effects
+				(font
+					(size 1.27 1.27)
+				)
+				(hide yes)
+			)
+		)
+		(property "Datasheet" ""
+			(at 109.22 115.57 0)
+			(effects
+				(font
+					(size 1.27 1.27)
+				)
+				(hide yes)
+			)
+		)
+		(property "Description" "Power symbol creates a global label with name \"GND\" , ground"
+			(at 109.22 115.57 0)
+			(effects
+				(font
+					(size 1.27 1.27)
+				)
+				(hide yes)
+			)
+		)
+		(pin "1"
+		)
+		(instances
+			(project "nrf24l01_pa_lna"
+				(path "/45a19bd1-4465-4728-867b-7ac302c76a0c"
+					(reference "#PWR049")
+					(unit 1)
+				)
+			)
+		)
+	)
+	(symbol
 		(lib_id "Device:R")
 		(at 57.15 81.28 90)
@@
 	)
 	(symbol
+		(lib_id "power:PWR_FLAG")
+		(at 109.22 113.03 0)
+		(unit 1)
+		(exclude_from_sim no)
+		(in_bom yes)
+		(on_board yes)
+		(dnp no)
+		(fields_autoplaced yes)
+		(property "Reference" "#FLG02"
+			(at 109.22 111.125 0)
+			(effects
+				(font
+					(size 1.27 1.27)
+				)
+				(hide yes)
+			)
+		)
+		(property "Value" "PWR_FLAG"
+			(at 109.22 107.95 0)
+			(effects
+				(font
+					(size 1.27 1.27)
+				)
+			)
+		)
+		(property "Footprint" ""
+			(at 109.22 113.03 0)
+			(effects
+				(font
+					(size 1.27 1.27)
+				)
+				(hide yes)
+			)
+		)
+		(property "Datasheet" "~"
+			(at 109.22 113.03 0)
+			(effects
+				(font
+					(size 1.27 1.27)
+				)
+				(hide yes)
+			)
+		)
+		(property "Description" "Special symbol for telling ERC where power comes from"
+			(at 109.22 113.03 0)
+			(effects
+				(font
+					(size 1.27 1.27)
+				)
+				(hide yes)
+			)
+		)
+		(pin "1"
+		)
+		(instances
+			(project "nrf24l01_pa_lna"
+				(path "/45a19bd1-4465-4728-867b-7ac302c76a0c"
+					(reference "#FLG02")
+					(unit 1)
+				)
+			)
+		)
+	)
+	(symbol
 		(lib_id "Device:R")
 		(at 92.71 140.97 90)
@@
 					(unit 1)
 				)
+			)
+		)
+	)
+	(symbol
+		(lib_id "power:PWR_FLAG")
+		(at 38.1 246.38 0)
+		(unit 1)
+		(exclude_from_sim no)
+		(in_bom yes)
+		(on_board yes)
+		(dnp no)
+		(fields_autoplaced yes)
+		(property "Reference" "#FLG01"
+			(at 38.1 244.475 0)
+			(effects
+				(font
+					(size 1.27 1.27)
+				)
+				(hide yes)
+			)
+		)
+		(property "Value" "PWR_FLAG"
+			(at 38.1 241.3 0)
+			(effects
+				(font
+					(size 1.27 1.27)
+				)
+			)
+		)
+		(property "Footprint" ""
+			(at 38.1 246.38 0)
+			(effects
+				(font
+					(size 1.27 1.27)
+				)
+				(hide yes)
+			)
+		)
+		(property "Datasheet" "~"
+			(at 38.1 246.38 0)
+			(effects
+				(font
+					(size 1.27 1.27)
+				)
+				(hide yes)
+			)
+		)
+		(property "Description" "Special symbol for telling ERC where power comes from"
+			(at 38.1 246.38 0)
+			(effects
+				(font
+					(size 1.27 1.27)
+				)
+				(hide yes)
+			)
+		)
+		(pin "1"
+		)
+		(instances
+			(project ""
+				(path "/45a19bd1-4465-4728-867b-7ac302c76a0c"
+					(reference "#FLG01")
+					(unit 1)
+				)

Commit message: Placing elements, making connections.
Parts:
- removed C25, C26, C27: 10n, Capacitor_SMD:C_0402_1005Metric, symbol Device:C
- U1: footprint Package_DFN_QFN:QFN-20-1EP_4x4mm_P0.5mm_EP2.5x2.5mm -> nrf24l01:QFN-20-4x4mm_P0.5mm_EP2.5x2.5mm

Commit message: Finished the design in bulk...
Parts:
- removed U3: MCP1802x-xx02xOT, Package_TO_SOT_SMD:SOT-23-5, symbol Regulator_Linear:MCP1802x-xx02xOT
- added U4: MCP1825S, Package_TO_SOT_SMD:SOT-223-3_TabPin2, symbol Regulator_Linear:MCP1825S
Connections:
- net GND: now also U4.2 (GND)
- net VDD: now also U4.3 (VO)
- net v_pwr: now also U4.1 (VI)
Other:
- moved on the sheet: C22
Changed lines of the file:
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@@
 	)
 	(junction
-		(at 54.61 248.92)
-		(diameter 0)
-		(color 0 0 0 0)
-	)
-	(junction
 		(at 222.25 152.4)
 		(diameter 0)
@@
 	)
 	(junction
-		(at 83.82 248.92)
+		(at 78.74 248.92)
 		(diameter 0)
 		(color 0 0 0 0)
@@
 	(wire
 		(pts
-			(xy 80.01 248.92) (xy 83.82 248.92)
+			(xy 74.93 248.92) (xy 78.74 248.92)
 		)
 		(stroke
@@
 	(wire
 		(pts
-			(xy 83.82 248.92) (xy 83.82 251.46)
+			(xy 78.74 248.92) (xy 78.74 251.46)
 		)
 		(stroke
@@
 	(wire
 		(pts
-			(xy 54.61 248.92) (xy 59.69 248.92)
+			(xy 38.1 248.92) (xy 59.69 248.92)
 		)
 		(stroke
@@
 	(wire
 		(pts
-			(xy 38.1 248.92) (xy 54.61 248.92)
-		)
-		(stroke
-			(width 0)
-			(type default)
-		)
-	)
-	(wire
-		(pts
 			(xy 346.71 93.98) (xy 368.3 93.98)
 		)
@@
 	(wire
 		(pts
-			(xy 59.69 251.46) (xy 54.61 251.46)
-		)
-		(stroke
-			(width 0)
-			(type default)
-		)
-	)
-	(wire
-		(pts
 			(xy 95.25 30.48) (xy 95.25 33.02)
 		)
@@
 	(wire
 		(pts
-			(xy 83.82 248.92) (xy 92.71 248.92)
+			(xy 78.74 248.92) (xy 87.63 248.92)
 		)
 		(stroke
@@
 	(wire
 		(pts
-			(xy 54.61 251.46) (xy 54.61 248.92)
-		)
-		(stroke
-			(width 0)
-			(type default)
-		)
-	)
-	(wire
-		(pts
 			(xy 95.25 40.64) (xy 95.25 43.18)
 		)
@@
 	(wire
 		(pts
-			(xy 69.85 259.08) (xy 69.85 261.62)
+			(xy 67.31 256.54) (xy 67.31 259.08)
 		)
 		(stroke
@@
 	(wire
 		(pts
-			(xy 83.82 259.08) (xy 83.82 261.62)
+			(xy 78.74 259.08) (xy 78.74 261.62)
 		)
 		(stroke
@@
 	(wire
 		(pts
-			(xy 92.71 248.92) (xy 92.71 246.38)
+			(xy 87.63 248.92) (xy 87.63 246.38)
 		)
 		(stroke
@@
 	(symbol
 		(lib_id "power:GND")
-		(at 69.85 261.62 0)
+		(at 67.31 259.08 0)
 		(unit 1)
 		(exclude_from_sim no)
@@
 		(dnp no)
 		(property "Reference" "#PWR043"
-			(at 69.85 267.97 0)
+			(at 67.31 265.43 0)
 			(effects
 				(font
@@
 		)
 		(property "Value" "GND"
-			(at 69.85 265.43 0)
+			(at 67.31 262.89 0)
 			(effects
 				(font
@@
 		)
 		(property "Footprint" ""
-			(at 69.85 261.62 0)
+			(at 67.31 259.08 0)
 			(effects
 				(font
@@
 		)
 		(property "Datasheet" ""
-			(at 69.85 261.62 0)
+			(at 67.31 259.08 0)
 			(effects
 				(font
@@
 		)
 		(property "Description" "Power symbol creates a global label with name \"GND\" , ground"
-			(at 69.85 261.62 0)
+			(at 67.31 259.08 0)
 			(effects
 				(font
@@
 	(symbol
 		(lib_id "power:GND")
-		(at 83.82 261.62 0)
+		(at 78.74 261.62 0)
 		(unit 1)
 		(exclude_from_sim no)
@@
 		(dnp no)
 		(property "Reference" "#PWR035"
-			(at 83.82 267.97 0)
+			(at 78.74 267.97 0)
 			(effects
 				(font
@@
 		)
 		(property "Value" "GND"
-			(at 83.82 265.43 0)
+			(at 78.74 265.43 0)
 			(effects
 				(font
@@
 		)
 		(property "Footprint" ""
-			(at 83.82 261.62 0)
+			(at 78.74 261.62 0)
 			(effects
 				(font
@@
 		)
 		(property "Datasheet" ""
-			(at 83.82 261.62 0)
+			(at 78.74 261.62 0)
 			(effects
 				(font
@@
 		)
 		(property "Description" "Power symbol creates a global label with name \"GND\" , ground"
-			(at 83.82 261.62 0)
+			(at 78.74 261.62 0)
 			(effects
 				(font
@@
 	)
 	(symbol
-		(lib_id "Regulator_Linear:MCP1802x-xx02xOT")
-		(at 69.85 251.46 0)
-		(unit 1)
-		(exclude_from_sim no)
-		(in_bom yes)
-		(on_board yes)
-		(dnp no)
-		(fields_autoplaced yes)
-		(property "Reference" "U3"
-			(at 69.85 241.3 0)
-			(effects
-				(font
-					(size 1.27 1.27)
-				)
-			)
-		)
-		(property "Value" "MCP1802x-xx02xOT"
-			(at 69.85 243.84 0)
-			(effects
-				(font
-					(size 1.27 1.27)
-				)
-			)
-		)
-		(property "Footprint" "Package_TO_SOT_SMD:SOT-23-5"
-			(at 63.5 242.57 0)
-			(effects
-				(font
-					(size 1.27 1.27)
-					(italic yes)
-				)
-				(justify left)
-				(hide yes)
-			)
-		)
-		(property "Datasheet" "http://ww1.microchip.com/downloads/en/DeviceDoc/22053C.pdf"
-			(at 69.85 254 0)
-			(effects
-				(font
-					(size 1.27 1.27)
-				)
-				(hide yes)
-			)
-		)
-		(property "Description" "150mA, Tiny CMOS LDO With Shutdown, Fixed Voltage, SOT-23-5"
-			(at 69.85 251.46 0)
-			(effects
-				(font
-					(size 1.27 1.27)
-				)
-				(hide yes)
-			)
-		)
-		(property "url" "https://www.digikey.com/en/products/detail/microchip-technology/MCP1802T-3302I-OT/1679144?s=N4IgjCBcpg7LBOKoDGUBmBDANgZwKYA0IA9lANriwAsYYArCALrEAOALlCAMrsBOASwB2AcxABfYgFoATMhBpI-AK5FSFEIybjJIOZEoBbFKzAAOAAxztQA"
-			(at 69.85 251.46 0)
-			(effects
-				(font
-					(size 1.27 1.27)
-				)
-				(hide yes)
-			)
-		)
-		(pin "1"
-		)
-		(pin "3"
-		)
-		(pin "2"
-		)
-		(pin "4"
-		)
-		(pin "5"
-		)
-		(instances
-			(project "nrf24l01_pa_lna"
-				(path "/45a19bd1-4465-4728-867b-7ac302c76a0c"
-					(reference "U3")
-					(unit 1)
-				)
-			)
-		)
-	)
-	(symbol
 		(lib_id "Device:C")
-		(at 83.82 255.27 0)
+		(at 78.74 255.27 0)
 		(unit 1)
 		(exclude_from_sim no)
@@
 		(dnp no)
 		(property "Reference" "C22"
-			(at 84.455 252.73 0)
+			(at 79.375 252.73 0)
 			(effects
 				(font
@@
 		)
 		(property "Value" "4u7"
-			(at 84.455 257.81 0)
+			(at 79.375 257.81 0)
 			(effects
 				(font
@@
 		)
 		(property "Footprint" "Capacitor_SMD:C_0603_1608Metric"
-			(at 84.7852 259.08 0)
+			(at 79.7052 259.08 0)
 			(effects
 				(font
@@
 		)
 		(property "Datasheet" "~"
-			(at 83.82 255.27 0)
+			(at 78.74 255.27 0)
 			(effects
 				(font
@@
 		)
 		(property "Description" "Unpolarized capacitor"
-			(at 83.82 255.27 0)
+			(at 78.74 255.27 0)
 			(effects
 				(font
@@
 		)
 		(property "url" "https://www.digikey.com/product-detail/en/samsung-electro-mechanics-america-inc/CL10B475KQ8NQNC/1276-2087-1-ND/3890173"
-			(at 83.82 255.27 0)
+			(at 78.74 255.27 0)
 			(effects
 				(font
@@
 	(symbol
 		(lib_id "power:VDD")
-		(at 92.71 246.38 0)
+		(at 87.63 246.38 0)
 		(unit 1)
 		(exclude_from_sim no)
@@
 		(fields_autoplaced yes)
 		(property "Reference" "#PWR036"
-			(at 92.71 250.19 0)
+			(at 87.63 250.19 0)
 			(effects
 				(font
@@
 		)
 		(property "Value" "VDD"
-			(at 92.71 241.3 0)
+			(at 87.63 241.3 0)
 			(effects
 				(font
@@
 		)
 		(property "Footprint" ""
-			(at 92.71 246.38 0)
+			(at 87.63 246.38 0)
 			(effects
 				(font
@@
 		)
 		(property "Datasheet" ""
-			(at 92.71 246.38 0)
+			(at 87.63 246.38 0)
 			(effects
 				(font
@@
 		)
 		(property "Description" "Power symbol creates a global label with name \"VDD\""
-			(at 92.71 246.38 0)
+			(at 87.63 246.38 0)
 			(effects
 				(font
@@
 					(unit 1)
 				)
+			)
+		)
+	)
+	(symbol
+		(lib_id "Regulator_Linear:MCP1825S")
+		(at 67.31 248.92 0)
+		(unit 1)
+		(exclude_from_sim no)
+		(in_bom yes)
+		(on_board yes)
+		(dnp no)
+		(fields_autoplaced yes)
+		(property "Reference" "U4"
+			(at 67.31 242.57 0)
+			(effects
+				(font
+					(size 1.27 1.27)
+				)
+			)
+		)
+		(property "Value" "MCP1825S"
+			(at 67.31 245.11 0)
+			(effects
+				(font
+					(size 1.27 1.27)
+				)
+			)
+		)
+		(property "Footprint" "Package_TO_SOT_SMD:SOT-223-3_TabPin2"
+			(at 64.77 245.11 0)
+			(effects
+				(font
+					(size 1.27 1.27)
+				)
+				(hide yes)
+			)
+		)
+		(property "Datasheet" "http://ww1.microchip.com/downloads/en/devicedoc/22056b.pdf"
+			(at 67.31 242.57 0)
+			(effects
+				(font
+					(size 1.27 1.27)
+				)
+				(hide yes)
+			)
+		)
+		(property "Description" "500mA, Low-Voltage, Low Quiescent Current LDO Regulator, SOT-223, TO-220, TO-263"
+			(at 67.31 248.92 0)
+			(effects
+				(font
+					(size 1.27 1.27)
+				)
+				(hide yes)
+			)
+		)
+		(property "url" "https://www.digikey.com/en/products/detail/microchip-technology/MCP1825S-3302E-DB/1636103?s=N4IgTCBcDaILIGEAKBGAHGArAZQLQGZ8AGMAUQHoARAIRAF0BfIA"
+			(at 67.31 248.92 0)
+			(effects
+				(font
+					(size 1.27 1.27)
+				)
+				(hide yes)
+			)
+		)
+		(pin "2"
+		)
+		(pin "3"
+		)
+		(pin "1"
+		)
+		(instances
+			(project ""
+				(path "/45a19bd1-4465-4728-867b-7ac302c76a0c"
+					(reference "U4")
+					(unit 1)
+				)
